File: rgb-matrix-pcb/rgb-matrix-pcb.kicad_pcb (KiCad board)
At the start: 2 copper layers, 81.3 x 76.2 mm, 36 parts, among them J1 Conn_01x16_Socket, J2 Conn_01x16_Socket, J3 Conn_01x05, U1 74HC595, U2 74HC595, U3 74HC595, U4 74HC595

Commit message: Added schematic notes for greenwired current amplifiers
Parts:
- C1, C2, C3, C4: value 0.1 -> 0.1u
- R1, R2, R3, R4, R5, R6, R7, R8: value 75 -> 33R
- R10, R11, R12, R13, R14, R15, R16, R9: value 75 -> 2R2
- R17, R18, R19, R20, R21, R22, R23, R24: value 75 -> 91R
